File: pcb/dongle.brd (EAGLE design)
At the start: 160 x 100 mm, 13 parts, among them IC1 ATSAMD21E18A-AFT, IC2 MCP73831T-2ACI/OT, IC3 IC_XC8107AC20MR-G

Commit message: Changed some parts sources and worked on board
Parts:
- removed JP1: (no value), pinhead:1X02
- removed USB: CX60-24S-UNIT, CX60-24S-UNIT:HIROSE_CX60-24S-UNIT
- added B4: EVP-BFAC1A000, EVP-BFAC1A000:EVPBFAC1A000
- added CN1: (no value), adafruit:JST-PH-2-SMT-RA
- added USB1: USB4155-03-C_REVA, USB4155-03-C_REVA:GCT_USB4155-03-C_REVA
- added USB2: 12401610E4#2A, 12401610E4_2A:AMPHENOL_12401610E4#2A
- B1, B2, B3: value FSM4JSMA -> EVP-BFAC1A000; device FSM4JSMA:FSM4JSMA -> EVP-BFAC1A000:EVPBFAC1A000
- moved B3 113.1 mm to (40.6, 17.8)
- moved B2 74.4 mm to (25.4, 17.8)
- moved IC3 69.9 mm to (6.35, -27.9)
- moved B1 69.3 mm to (10.2, 17.8)
- moved IC2 68.5 mm to (7.62, -17.8)
- moved IC1 38.6 mm to (11.4, 6.35)
Connections:
- net N$3 renamed 3.3V
- net N$4 renamed STAT
- net N$5 renamed PROG
- removed net N$1: IC2.3, JP1.1
- removed net N$2: C1.2, IC2.4, IC3.CE, IC3.G0, IC3.VIN, USB.A4, USB.A9, USB.B4, USB.B9
- new net 3.3VBAT: CN1.1, IC2.3
- new net 5VIN: C1.2, IC2.4, IC3.CE, IC3.G0, IC3.VIN, USB1.A4, USB1.A9, USB1.B4, USB1.B9, USB2.A4, USB2.A9, USB2.B4, USB2.B9
- new net B: IC1.8, LED1.3
- new net G: IC1.7, LED1.2
- new net R: IC1.6, LED1.1
- net CC: now also USB1.A5, USB2.A5, USB2.B5; no longer USB.A5
- net D+: now also USB1.A6, USB2.A6, USB2.B6; no longer USB.A6
- net D-: now also USB1.A7, USB2.A7, USB2.B7; no longer USB.A7
- net GND: now also CN1.2, LED1.4, USB1.A1, USB1.A12, USB1.B1, USB1.B12, USB1.S1, USB1.S2, USB2.A1, USB2.A12, USB2.B1, USB2.B12, USB2.S1, USB2.S2, USB2.S3, USB2.S4; no longer JP1.2, USB.A1, USB.A12, USB.B1, USB.B12, USB.S1, USB.S2, USB.S3, USB.S4
Routing:
- net GND: track 0.00 -> 1.56 mm
- added copper zone on layer 1, net GND
- added copper zone on layer 16, net GND
Other:
- board size 160 x 100 mm -> 50.8 x 34.3 mm
