File: pcb/dongle.sch (EAGLE design)
At the start: 11 parts, among them IC1 ATSAMD21E18A-AFT, IC2 MCP73831T-2ACI/OT, IC3 IC_XC8107AC20MR-G

Commit message: Lots of all around work on the code and board
Parts:
- removed S2: FSM4JSMA, FSM4JSMA:FSM4JSMA
- added B1, B3: FSM4JSMA, FSM4JSMA:FSM4JSMA
- added R3: (no value), rcl:R-US_R0805
- LED1: value SMD-LX5050RGB-TR -> ASMB-MTB1-0B3A2; device SMD-LX5050RGB-TR:SMD-LX5050RGB-TR -> SamacSys_Parts:ASMB-MTB1-0B3A2
- renumbered S1 to B2
Connections:
- new net CC: R3.1, USB.CC
- net GND: now also R3.2
Other:
- moved on the sheet: C1, IC2, IC3, JP1, R1, R2, USB

Commit message: Changed some parts sources and worked on board
Parts:
- removed JP1: (no value), pinhead:PINHD-1X2
- removed USB: CX60-24S-UNIT, CX60-24S-UNIT:CX60-24S-UNIT
- added B4: EVP-BFAC1A000, EVP-BFAC1A000:EVP-BFAC1A000
- added CN1: (no value), adafruit:JST_2PIN-SMT-RA
- added USB1: USB4155-03-C_REVA, USB4155-03-C_REVA:USB4155-03-C_REVA
- added USB2: 12401610E4#2A, 12401610E4_2A:12401610E4#2A
- B1, B2, B3: value FSM4JSMA -> EVP-BFAC1A000; device FSM4JSMA:FSM4JSMA -> EVP-BFAC1A000:EVP-BFAC1A000
Connections:
- net N$3 renamed 3.3V
- net N$4 renamed STAT
- net N$5 renamed PROG
- removed net N$1: IC2.VBAT, JP1.1
- removed net N$2: C1.2, IC2.VDD, IC3.CE, IC3.GO, IC3.VIN, USB.VBUS_A, USB.VBUS_B
- new net 3.3VBAT: CN1.2, IC2.VBAT
- new net 5VIN: C1.2, IC2.VDD, IC3.CE, IC3.GO, IC3.VIN, USB1.VBUS_A, USB1.VBUS_B, USB2.VBUS_A4, USB2.VBUS_A9, USB2.VBUS_B4, USB2.VBUS_B9
- new net B: IC1.PA07, LED1.K_(BLUE)
- new net G: IC1.PA06, LED1.K_(GREEN)
- new net R: IC1.PA05, LED1.K_(RED)
- net CC: now also USB1.CC1, USB2.CC1, USB2.CC2; no longer USB.CC
- net D+: now also USB1.DP1, USB2.DA+, USB2.DB+; no longer USB.D+
- net D-: now also USB1.DN1, USB2.DA-, USB2.DB-; no longer USB.D-
- net GND: now also CN1.1, LED1.COM_A, USB1.GND_A, USB1.GND_B, USB1.SHELL_GND, USB2.GND_A1, USB2.GND_A12, USB2.GND_B1, USB2.GND_B12, USB2.SHIELD; no longer JP1.2, USB.GNDA, USB.GNDB, USB.SHIELD1, USB.SHIELD2
Other:
- moved on the sheet: B1, B2, B3, LED1, R2
